File: blinksy-solo.kicad_pcb (KiCad board)
At the start: 2 copper layers, 69.8 x 50.8 mm, 26 parts, among them P1 D1, P10 PWR, P2 D2, P3 D3, P4 D4, P5 D5, P6 D6, P7 D7, P8 D8, P9 AUX_DATA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

Commit message: Bump rev to 2, drop issue date
Parts:
- removed M** (x2): 3mm MNT, sinistral:3mmMNT
- added REF**: MountingHole_3.5mm_Pad, Mounting_Holes:MountingHole_3.5mm_Pad, F.Cu at (175.3, 86.4)
- added REF**: MountingHole_3.5mm_Pad, Mounting_Holes:MountingHole_3.5mm_Pad, F.Cu at (139.7, 115.6)
- moved P9 1.27 mm to (130.8, 109.2)
- moved U1 1.27 mm to (167.6, 108.0)
Routing:
- net /OCTO2: track 46.8 -> 43.7 mm
- net /OCTO4: track 31.4 -> 33.9 mm
- net /OCTO5: track 26.3 -> 28.9 mm
- net /OCTO3: track 28.9 -> 31.4 mm
- net VCC: track 179.3 -> 177.3 mm
- net /AUX2: track 22.4 -> 20.6 mm
- net /AUX3: track 26.0 -> 24.2 mm
- net /AUX5: track 38.3 -> 37.5 mm
- net /AUX1: track 18.8 -> 18.2 mm
- net /OCTO6: track 24.7 -> 24.2 mm
- net /OCTO7: track 21.2 -> 20.6 mm
- net /OCTO8: track 26.9 -> 27.4 mm
- net /OCTO1: track 16.1 -> 15.5 mm
